Commit message: EDIT: Fixed install errors

File: urdf/locobot.urdf.xacro (robot description, xacro)
@@ -13,5 +13,5 @@
   <xacro:property name="pi_offset" value="0.00001"/>
   <xacro:if value="$(arg load_gazebo_configs)">
-    <xacro:include filename="$(find interbotix_xslocobot_gazebo)/config/locobot_configs.gazebo"/>
+    <xacro:include filename="$(find locobot_simulation)/config/locobot_configs.gazebo"/>
   </xacro:if>
   <xacro:if value="${urdf_loc != ''}">
@@ -19,5 +19,5 @@
   </xacro:if>
   <material name="interbotix_black">
-    <texture filename="package://interbotix_xslocobot_descriptions/meshes/interbotix_black.png"/>
+    <texture filename="package://locobot_simulation/meshes/interbotix_black.png"/>
   </material>
     <!-- ********************************** Kobuki ********************************** -->
@@ -32,5 +32,5 @@
       <origin rpy="0 0 0" xyz="0.001 0 0.05199"/>
       <geometry>
-        <mesh filename="package://interbotix_xslocobot_descriptions/meshes/locobot_meshes/locobot_main_body.dae"/>
+        <mesh filename="package://locobot_simulation/meshes/locobot_meshes/locobot_main_body.dae"/>
       </geometry>
     </visual>
@@ -66,5 +66,5 @@
       <origin rpy="0 0 0" xyz="0 0 0"/>
       <geometry>
-        <mesh filename="package://interbotix_xslocobot_descriptions/meshes/locobot_meshes/locobot_wheel.dae"/>
+        <mesh filename="package://locobot_simulation/meshes/locobot_meshes/locobot_wheel.dae"/>
       </geometry>
     </visual>
@@ -100,5 +100,5 @@
       <origin rpy="0 0 0" xyz="0 0 0"/>
       <geometry>
-        <mesh filename="package://interbotix_xslocobot_descriptions/meshes/locobot_meshes/locobot_wheel.dae"/>
+        <mesh filename="package://locobot_simulation/meshes/locobot_meshes/locobot_wheel.dae"/>
       </geometry>
     </visual>
@@ -209,5 +209,5 @@
       <origin rpy="0 0 0" xyz="0 0 0"/>
       <geometry>
-        <mesh filename="package://interbotix_xslocobot_descriptions/meshes/locobot_meshes/locobot_base_plate.stl" scale="0.001 0.001 0.001"/>
+        <mesh filename="package://locobot_simulation/meshes/locobot_meshes/locobot_base_plate.stl" scale="0.001 0.001 0.001"/>
       </geometry>
       <material name="interbotix_black"/>
@@ -216,5 +216,5 @@
       <origin rpy="0 0 0" xyz="0 0 0"/>
       <geometry>
-        <mesh filename="package://interbotix_xslocobot_descriptions/meshes/locobot_meshes/locobot_base_plate.stl" scale="0.001 0.001 0.001"/>
+        <mesh filename="package://locobot_simulation/meshes/locobot_meshes/locobot_base_plate.stl" scale="0.001 0.001 0.001"/>
       </geometry>
     </collision>
@@ -226,5 +226,5 @@
   </link>
   <xacro:if value="${arm_type != 'mobile_base'}">
-    <xacro:include filename="$(find interbotix_xslocobot_descriptions)/urdf/$(arg arm_model).urdf.xacro"/>
+    <xacro:include filename="$(find locobot_simulation)/urdf/$(arg arm_model).urdf.xacro"/>
     <xacro:if value="${arm_type == 'mobile_wx200'}">
       <joint name="arm_cradle" type="fixed">
@@ -238,5 +238,5 @@
          <origin rpy="0 0 0" xyz="0 0 0"/>
          <geometry>
-           <mesh filename="package://interbotix_xslocobot_descriptions/meshes/locobot_meshes/locobot_arm_cradle.stl" scale="0.001 0.001 0.001"/>
+           <mesh filename="package://locobot_simulation/meshes/locobot_meshes/locobot_arm_cradle.stl" scale="0.001 0.001 0.001"/>
          </geometry>
          <material name="interbotix_black"/>
@@ -245,5 +245,5 @@
          <origin rpy="0 0 0" xyz="0 0 0"/>
          <geometry>
-           <mesh filename="package://interbotix_xslocobot_descriptions/meshes/locobot_meshes/locobot_arm_cradle.stl" scale="0.001 0.001 0.001"/>
+           <mesh filename="package://locobot_simulation/meshes/locobot_meshes/locobot_arm_cradle.stl" scale="0.001 0.001 0.001"/>
          </geometry>
        </collision>
@@ -266,5 +266,5 @@
       <origin rpy="0 0 0" xyz="0 0 0"/>
       <geometry>
-        <mesh filename="package://interbotix_xslocobot_descriptions/meshes/locobot_meshes/locobot_battery.stl" scale="0.001 0.001 0.001"/>
+        <mesh filename="package://locobot_simulation/meshes/locobot_meshes/locobot_battery.stl" scale="0.001 0.001 0.001"/>
       </geometry>
       <material name="">
@@ -275,5 +275,5 @@
       <origin rpy="0 0 0" xyz="0 0 0"/>
       <geometry>
-        <mesh filename="package://interbotix_xslocobot_descriptions/meshes/locobot_meshes/locobot_battery.stl" scale="0.001 0.001 0.001"/>
+        <mesh filename="package://locobot_simulation/meshes/locobot_meshes/locobot_battery.stl" scale="0.001 0.001 0.001"/>
       </geometry>
     </collision>
@@ -295,5 +295,5 @@
         <origin rpy="0 0 0" xyz="0 0 0"/>
         <geometry>
-          <mesh filename="package://interbotix_xslocobot_descriptions/meshes/locobot_meshes/locobot_camera_tower_large.stl" scale="0.001 0.001 0.001"/>
+          <mesh filename="package://locobot_simulation/meshes/locobot_meshes/locobot_camera_tower_large.stl" scale="0.001 0.001 0.001"/>
         </geometry>
         <material name="interbotix_black"/>
@@ -302,5 +302,5 @@
         <origin rpy="0 0 0" xyz="0 0 0"/>
         <geometry>
-          <mesh filename="package://interbotix_xslocobot_descriptions/meshes/locobot_meshes/locobot_camera_tower_large_simple.stl" scale="0.001 0.001 0.001"/>
+          <mesh filename="package://locobot_simulation/meshes/locobot_meshes/locobot_camera_tower_large_simple.stl" scale="0.001 0.001 0.001"/>
         </geometry>
       </collision>
@@ -317,5 +317,5 @@
         <origin rpy="0 0 0" xyz="0 0 0"/>
         <geometry>
-          <mesh filename="package://interbotix_xslocobot_descriptions/meshes/locobot_meshes/locobot_camera_tower_small.stl" scale="0.001 0.001 0.001"/>
+          <mesh filename="package://locobot_simulation/meshes/locobot_meshes/locobot_camera_tower_small.stl" scale="0.001 0.001 0.001"/>
         </geometry>
         <material name="interbotix_black"/>
@@ -324,5 +324,5 @@
         <origin rpy="0 0 0" xyz="0 0 0"/>
         <geometry>
-          <mesh filename="package://interbotix_xslocobot_descriptions/meshes/locobot_meshes/locobot_camera_tower_small_simple.stl" scale="0.001 0.001 0.001"/>
+          <mesh filename="package://locobot_simulation/meshes/locobot_meshes/locobot_camera_tower_small_simple.stl" scale="0.001 0.001 0.001"/>
         </geometry>
       </collision>
@@ -360,5 +360,5 @@
       <origin rpy="0 0 ${pi/2}" xyz="0 0 0"/>
       <geometry>
-        <mesh filename="package://interbotix_xslocobot_descriptions/meshes/locobot_meshes/locobot_pan.stl" scale="0.001 0.001 0.001"/>
+        <mesh filename="package://locobot_simulation/meshes/locobot_meshes/locobot_pan.stl" scale="0.001 0.001 0.001"/>
       </geometry>
       <material name="interbotix_black"/>
@@ -367,5 +367,5 @@
       <origin rpy="0 0 ${pi/2}" xyz="0 0 0"/>
       <geometry>
-        <mesh filename="package://interbotix_xslocobot_descriptions/meshes/locobot_meshes/locobot_pan.stl" scale="0.001 0.001 0.001"/>
+        <mesh filename="package://locobot_simulation/meshes/locobot_meshes/locobot_pan.stl" scale="0.001 0.001 0.001"/>
       </geometry>
     </collision>
@@ -396,5 +396,5 @@
       <origin rpy="0 0 ${pi/2}" xyz="0 0 0"/>
       <geometry>
-        <mesh filename="package://interbotix_xslocobot_descriptions/meshes/locobot_meshes/locobot_tilt.stl" scale="0.001 0.001 0.001"/>
+        <mesh filename="package://locobot_simulation/meshes/locobot_meshes/locobot_tilt.stl" scale="0.001 0.001 0.001"/>
       </geometry>
       <material name="interbotix_black"/>
@@ -403,5 +403,5 @@
       <origin rpy="0 0 ${pi/2}" xyz="0 0 0"/>
       <geometry>
-        <mesh filename="package://interbotix_xslocobot_descriptions/meshes/locobot_meshes/locobot_tilt.stl" scale="0.001 0.001 0.001"/>
+        <mesh filename="package://locobot_simulation/meshes/locobot_meshes/locobot_tilt.stl" scale="0.001 0.001 0.001"/>
       </geometry>
     </collision>
@@ -421,5 +421,5 @@
       <origin rpy="0 0 0" xyz="0 0 0"/>
       <geometry>
-        <mesh filename="package://interbotix_xslocobot_descriptions/meshes/locobot_meshes/locobot_camera.stl" scale="0.001 0.001 0.001"/>
+        <mesh filename="package://locobot_simulation/meshes/locobot_meshes/locobot_camera.stl" scale="0.001 0.001 0.001"/>
       </geometry>
       <material name="">
@@ -430,5 +430,5 @@
       <origin rpy="0 0 0" xyz="0 0 0"/>
       <geometry>
-        <mesh filename="package://interbotix_xslocobot_descriptions/meshes/locobot_meshes/locobot_camera.stl" scale="0.001 0.001 0.001"/>
+        <mesh filename="package://locobot_simulation/meshes/locobot_meshes/locobot_camera.stl" scale="0.001 0.001 0.001"/>
       </geometry>
     </collision>
@@ -448,5 +448,5 @@
       <origin rpy="0 0 0" xyz="0 0 0"/>
       <geometry>
-        <mesh filename="package://interbotix_xslocobot_descriptions/meshes/locobot_meshes/locobot_camera.stl" scale="0.001 0.001 0.001"/>
+        <mesh filename="package://locobot_simulation/meshes/locobot_meshes/locobot_camera.stl" scale="0.001 0.001 0.001"/>
       </geometry>
       <material name="">
@@ -457,5 +457,5 @@
       <origin rpy="0 0 0" xyz="0 0 0"/>
       <geometry>
-        <mesh filename="package://interbotix_xslocobot_descriptions/meshes/locobot_meshes/locobot_camera.stl" scale="0.001 0.001 0.001"/>
+        <mesh filename="package://locobot_simulation/meshes/locobot_meshes/locobot_camera.stl" scale="0.001 0.001 0.001"/>
       </geometry>
     </collision>
@@ -482,5 +482,5 @@
         <origin rpy="0 0 0" xyz="0 0 0"/>
         <geometry>
-          <mesh filename="package://interbotix_xslocobot_descriptions/meshes/locobot_meshes/locobot_lidar_tower.stl" scale="0.001 0.001 0.001"/>
+          <mesh filename="package://locobot_simulation/meshes/locobot_meshes/locobot_lidar_tower.stl" scale="0.001 0.001 0.001"/>
         </geometry>
         <material name="interbotix_black"/>
@@ -489,5 +489,5 @@
         <origin rpy="0 0 0" xyz="0 0 0"/>
         <geometry>
-          <mesh filename="package://interbotix_xslocobot_descriptions/meshes/locobot_meshes/locobot_lidar_tower_simple.stl" scale="0.001 0.001 0.001"/>
+          <mesh filename="package://locobot_simulation/meshes/locobot_meshes/locobot_lidar_tower_simple.stl" scale="0.001 0.001 0.001"/>
         </geometry>
       </collision>
@@ -507,5 +507,5 @@
         <origin rpy="0 0 0" xyz="0 0 0"/>
         <geometry>
-          <mesh filename="package://interbotix_xslocobot_descriptions/meshes/locobot_meshes/locobot_lidar.stl" scale="0.001 0.001 0.001"/>
+          <mesh filename="package://locobot_simulation/meshes/locobot_meshes/locobot_lidar.stl" scale="0.001 0.001 0.001"/>
         </geometry>
         <material name="interbotix_black"/>

File: urdf/mobile_wx250s.urdf.xacro (robot description, xacro)
@@ -11,5 +11,5 @@
       <origin rpy="${pi/2} 0 ${pi/2}" xyz="-0.095773 0 -0.10565023"/>
       <geometry>
-        <mesh filename="package://interbotix_xslocobot_descriptions/meshes/mobile_wx250s_meshes/mobile_wx250s_1_base.stl" scale="0.001 0.001 0.001"/>
+        <mesh filename="package://locobot_simulation/meshes/mobile_wx250s_meshes/mobile_wx250s_1_base.stl" scale="0.001 0.001 0.001"/>
       </geometry>
       <material name="interbotix_black"/>
@@ -18,5 +18,5 @@
       <origin rpy="${pi/2} 0 ${pi/2}" xyz="-0.095773 0 -0.10565023"/>
       <geometry>
-        <mesh filename="package://interbotix_xslocobot_descriptions/meshes/mobile_wx250s_meshes/mobile_wx250s_1_base.stl" scale="0.001 0.001 0.001"/>
+        <mesh filename="package://locobot_simulation/meshes/mobile_wx250s_meshes/mobile_wx250s_1_base.stl" scale="0.001 0.001 0.001"/>
       </geometry>
     </collision>
@@ -48,5 +48,5 @@
       <origin rpy="0 0 ${pi/2}" xyz="0 0 -0.003"/>
       <geometry>
-        <mesh filename="package://interbotix_xslocobot_descriptions/meshes/mobile_wx250s_meshes/mobile_wx250s_2_shoulder.stl" scale="0.001 0.001 0.001"/>
+        <mesh filename="package://locobot_simulation/meshes/mobile_wx250s_meshes/mobile_wx250s_2_shoulder.stl" scale="0.001 0.001 0.001"/>
       </geometry>
       <material name="interbotix_black"/>
@@ -55,5 +55,5 @@
       <origin rpy="0 0 ${pi/2}" xyz="0 0 -0.003"/>
       <geometry>
-        <mesh filename="package://interbotix_xslocobot_descriptions/meshes/mobile_wx250s_meshes/mobile_wx250s_2_shoulder.stl" scale="0.001 0.001 0.001"/>
+        <mesh filename="package://locobot_simulation/meshes/mobile_wx250s_meshes/mobile_wx250s_2_shoulder.stl" scale="0.001 0.001 0.001"/>
       </geometry>
     </collision>
@@ -85,5 +85,5 @@
       <origin rpy="0 0 ${pi/2}" xyz="0 0 0"/>
       <geometry>
-        <mesh filename="package://interbotix_xslocobot_descriptions/meshes/mobile_wx250s_meshes/mobile_wx250s_3_upper_arm.stl" scale="0.001 0.001 0.001"/>
+        <mesh filename="package://locobot_simulation/meshes/mobile_wx250s_meshes/mobile_wx250s_3_upper_arm.stl" scale="0.001 0.001 0.001"/>
       </geometry>
       <material name="interbotix_black"/>
@@ -92,5 +92,5 @@
       <origin rpy="0 0 ${pi/2}" xyz="0 0 0"/>
       <geometry>
-        <mesh filename="package://interbotix_xslocobot_descriptions/meshes/mobile_wx250s_meshes/mobile_wx250s_3_upper_arm.stl" scale="0.001 0.001 0.001"/>
+        <mesh filename="package://locobot_simulation/meshes/mobile_wx250s_meshes/mobile_wx250s_3_upper_arm.stl" scale="0.001 0.001 0.001"/>
       </geometry>
     </collision>
@@ -122,5 +122,5 @@
       <origin rpy="0 0 0" xyz="0 0 0"/>
       <geometry>
-        <mesh filename="package://interbotix_xslocobot_descriptions/meshes/mobile_wx250s_meshes/mobile_wx250s_4_upper_forearm.stl" scale="0.001 0.001 0.001"/>
+        <mesh filename="package://locobot_simulation/meshes/mobile_wx250s_meshes/mobile_wx250s_4_upper_forearm.stl" scale="0.001 0.001 0.001"/>
       </geometry>
       <material name="interbotix_black"/>
@@ -129,5 +129,5 @@
       <origin rpy="0 0 0" xyz="0 0 0"/>
       <geometry>
-        <mesh filename="package://interbotix_xslocobot_descriptions/meshes/mobile_wx250s_meshes/mobile_wx250s_4_upper_forearm.stl" scale="0.001 0.001 0.001"/>
+        <mesh filename="package://locobot_simulation/meshes/mobile_wx250s_meshes/mobile_wx250s_4_upper_forearm.stl" scale="0.001 0.001 0.001"/>
       </geometry>
     </collision>
@@ -159,5 +159,5 @@
       <origin rpy="${pi} 0 0" xyz="0 0 0"/>
       <geometry>
-        <mesh filename="package://interbotix_xslocobot_descriptions/meshes/mobile_wx250s_meshes/mobile_wx250s_5_lower_forearm.stl" scale="0.001 0.001 0.001"/>
+        <mesh filename="package://locobot_simulation/meshes/mobile_wx250s_meshes/mobile_wx250s_5_lower_forearm.stl" scale="0.001 0.001 0.001"/>
       </geometry>
       <material name="interbotix_black"/>
@@ -166,5 +166,5 @@
       <origin rpy="${pi} 0 0" xyz="0 0 0"/>
       <geometry>
-        <mesh filename="package://interbotix_xslocobot_descriptions/meshes/mobile_wx250s_meshes/mobile_wx250s_5_lower_forearm.stl" scale="0.001 0.001 0.001"/>
+        <mesh filename="package://locobot_simulation/meshes/mobile_wx250s_meshes/mobile_wx250s_5_lower_forearm.stl" scale="0.001 0.001 0.001"/>
       </geometry>
     </collision>
@@ -196,5 +196,5 @@
       <origin rpy="0 0 ${pi/2}" xyz="0 0 0"/>
       <geometry>
-        <mesh filename="package://interbotix_xslocobot_descriptions/meshes/mobile_wx250s_meshes/mobile_wx250s_6_wrist.stl" scale="0.001 0.001 0.001"/>
+        <mesh filename="package://locobot_simulation/meshes/mobile_wx250s_meshes/mobile_wx250s_6_wrist.stl" scale="0.001 0.001 0.001"/>
       </geometry>
       <material name="interbotix_black"/>
@@ -203,5 +203,5 @@
       <origin rpy="0 0 ${pi/2}" xyz="0 0 0"/>
       <geometry>
-        <mesh filename="package://interbotix_xslocobot_descriptions/meshes/mobile_wx250s_meshes/mobile_wx250s_6_wrist.stl" scale="0.001 0.001 0.001"/>
+        <mesh filename="package://locobot_simulation/meshes/mobile_wx250s_meshes/mobile_wx250s_6_wrist.stl" scale="0.001 0.001 0.001"/>
       </geometry>
     </collision>
@@ -233,5 +233,5 @@
       <origin rpy="0 0 ${pi/2}" xyz="-0.02 0 0"/>
       <geometry>
-        <mesh filename="package://interbotix_xslocobot_descriptions/meshes/mobile_wx250s_meshes/mobile_wx250s_7_gripper.stl" scale="0.001 0.001 0.001"/>
+        <mesh filename="package://locobot_simulation/meshes/mobile_wx250s_meshes/mobile_wx250s_7_gripper.stl" scale="0.001 0.001 0.001"/>
       </geometry>
       <material name="interbotix_black"/>
@@ -240,5 +240,5 @@
       <origin rpy="0 0 ${pi/2}" xyz="-0.02 0 0"/>
       <geometry>
-        <mesh filename="package://interbotix_xslocobot_descriptions/meshes/mobile_wx250s_meshes/mobile_wx250s_7_gripper.stl" scale="0.001 0.001 0.001"/>
+        <mesh filename="package://locobot_simulation/meshes/mobile_wx250s_meshes/mobile_wx250s_7_gripper.stl" scale="0.001 0.001 0.001"/>
       </geometry>
     </collision>
@@ -282,5 +282,5 @@
       <origin rpy="0 0 ${pi/2}" xyz="-0.0685 0 0"/>
       <geometry>
-        <mesh filename="package://interbotix_xslocobot_descriptions/meshes/mobile_wx250s_meshes/mobile_wx250s_8_gripper_prop.stl" scale="0.001 0.001 0.001"/>
+        <mesh filename="package://locobot_simulation/meshes/mobile_wx250s_meshes/mobile_wx250s_8_gripper_prop.stl" scale="0.001 0.001 0.001"/>
       </geometry>
       <material name="interbotix_black"/>
@@ -289,5 +289,5 @@
       <origin rpy="0 0 ${pi/2}" xyz="-0.0685 0 0"/>
       <geometry>
-        <mesh filename="package://interbotix_xslocobot_descriptions/meshes/mobile_wx250s_meshes/mobile_wx250s_8_gripper_prop.stl" scale="0.001 0.001 0.001"/>
+        <mesh filename="package://locobot_simulation/meshes/mobile_wx250s_meshes/mobile_wx250s_8_gripper_prop.stl" scale="0.001 0.001 0.001"/>
       </geometry>
     </collision>
@@ -308,5 +308,5 @@
       <origin rpy="0 0 0" xyz="0 0 0"/>
       <geometry>
-        <mesh filename="package://interbotix_xslocobot_descriptions/meshes/mobile_wx250s_meshes/mobile_wx250s_11_ar_tag.stl" scale="0.001 0.001 0.001"/>
+        <mesh filename="package://locobot_simulation/meshes/mobile_wx250s_meshes/mobile_wx250s_11_ar_tag.stl" scale="0.001 0.001 0.001"/>
       </geometry>
       <material name="interbotix_black"/>
@@ -315,5 +315,5 @@
       <origin rpy="0 0 0" xyz="0 0 0"/>
       <geometry>
-        <mesh filename="package://interbotix_xslocobot_descriptions/meshes/mobile_wx250s_meshes/mobile_wx250s_11_ar_tag.stl" scale="0.001 0.001 0.001"/>
+        <mesh filename="package://locobot_simulation/meshes/mobile_wx250s_meshes/mobile_wx250s_11_ar_tag.stl" scale="0.001 0.001 0.001"/>
       </geometry>
     </collision>
@@ -336,5 +336,5 @@
         <origin rpy="0 0 ${pi/2}" xyz="-0.063 0 0"/>
         <geometry>
-          <mesh filename="package://interbotix_xslocobot_descriptions/meshes/mobile_wx250s_meshes/mobile_wx250s_9_gripper_bar.stl" scale="0.001 0.001 0.001"/>
+          <mesh filename="package://locobot_simulation/meshes/mobile_wx250s_meshes/mobile_wx250s_9_gripper_bar.stl" scale="0.001 0.001 0.001"/>
         </geometry>
         <material name="interbotix_black"/>
@@ -343,5 +343,5 @@
         <origin rpy="0 0 ${pi/2}" xyz="-0.063 0 0"/>
         <geometry>
-          <mesh filename="package://interbotix_xslocobot_descriptions/meshes/mobile_wx250s_meshes/mobile_wx250s_9_gripper_bar.stl" scale="0.001 0.001 0.001"/>
+          <mesh filename="package://locobot_simulation/meshes/mobile_wx250s_meshes/mobile_wx250s_9_gripper_bar.stl" scale="0.001 0.001 0.001"/>
         </geometry>
       </collision>
@@ -387,5 +387,5 @@
           <origin rpy="${pi} ${pi} 0" xyz="0 0.005 0"/>
           <geometry>
-            <mesh filename="package://interbotix_xslocobot_descriptions/meshes/mobile_wx250s_meshes/mobile_wx250s_10_gripper_finger.stl" scale="0.001 0.001 0.001"/>
+            <mesh filename="package://locobot_simulation/meshes/mobile_wx250s_meshes/mobile_wx250s_10_gripper_finger.stl" scale="0.001 0.001 0.001"/>
           </geometry>
           <material name="interbotix_black"/>
@@ -394,5 +394,5 @@
           <origin rpy="${pi} ${pi} 0" xyz="0 0.005 0"/>
           <geometry>
-            <mesh filename="package://interbotix_xslocobot_descriptions/meshes/mobile_wx250s_meshes/mobile_wx250s_10_gripper_finger.stl" scale="0.001 0.001 0.001"/>
+            <mesh filename="package://locobot_simulation/meshes/mobile_wx250s_meshes/mobile_wx250s_10_gripper_finger.stl" scale="0.001 0.001 0.001"/>
           </geometry>
         </collision>
@@ -427,5 +427,5 @@
           <origin rpy="0 ${pi} 0" xyz="0 -0.005 0"/>
           <geometry>
-            <mesh filename="package://interbotix_xslocobot_descriptions/meshes/mobile_wx250s_meshes/mobile_wx250s_10_gripper_finger.stl" scale="0.001 0.001 0.001"/>
+            <mesh filename="package://locobot_simulation/meshes/mobile_wx250s_meshes/mobile_wx250s_10_gripper_finger.stl" scale="0.001 0.001 0.001"/>
           </geometry>
           <material name="interbotix_black"/>
@@ -434,5 +434,5 @@
           <origin rpy="0 ${pi} 0" xyz="0 -0.005 0"/>
           <geometry>
-            <mesh filename="package://interbotix_xslocobot_descriptions/meshes/mobile_wx250s_meshes/mobile_wx250s_10_gripper_finger.stl" scale="0.001 0.001 0.001"/>
+            <mesh filename="package://locobot_simulation/meshes/mobile_wx250s_meshes/mobile_wx250s_10_gripper_finger.stl" scale="0.001 0.001 0.001"/>
           </geometry>
         </collision>
