Commit message: ADD: YoloV5 - ugly but works

File: urdf/locobot.urdf.xacro (robot description, xacro)
@@ -469,10 +469,5 @@
   <xacro:if value="$(arg show_lidar)">
     <joint name="lidar_tower" type="fixed">
-      <xacro:if value="${arm_type == 'mobile_wx250s'}">
-        <origin rpy="0 0 0" xyz="-0.074 0 0.44425"/>
-      </xacro:if>
-      <xacro:unless value="${arm_type == 'mobile_wx250s'}">
-        <origin rpy="0 0 0" xyz="-0.074 0 0.38425"/>
-      </xacro:unless>
+      <xacro:insert_block name="origin"/>
       <parent link="$(arg robot_name)/camera_tower_link"/>
       <child link="$(arg robot_name)/lidar_tower_link"/>
@@ -498,4 +493,10 @@
       </inertial>
     </link>
+    <gazebo reference="$(arg robot_name)/lidar_tower_link">
+      <material>Custom/Interbotix</material>
+    </gazebo>
+    <gazebo reference="lidar_tower">
+      <disableFixedJointLumping>true</disableFixedJointLumping>
+    </gazebo>
     <joint name="lidar" type="fixed">
       <origin rpy="0 0 ${pi}" xyz="0 0 0.09425"/>
@@ -503,4 +504,7 @@
       <child link="$(arg robot_name)/laser_frame_link"/>
     </joint>
+    <gazebo reference="lidar">
+      <disableFixedJointLumping>true</disableFixedJointLumping>
+    </gazebo>
     <link name="$(arg robot_name)/laser_frame_link">
       <visual>
@@ -523,4 +527,36 @@
       </inertial>
     </link>
+    <gazebo reference="$(arg robot_name)/laser_frame_link">
+      <material>Custom/Interbotix</material>
+      <sensor type="ray" name="rplidar">
+        <pose>0 0 0 0 0 0</pose>
+        <visualize>false</visualize>
+        <update_rate>30</update_rate>
+        <ray>
+          <scan>
+            <horizontal>
+              <samples>400</samples>
+              <resolution>1</resolution>
+              <min_angle>-3.14159</min_angle>
+              <max_angle>3.14159</max_angle>
+            </horizontal>
+          </scan>
+          <range>
+            <min>0.2</min>
+            <max>16.0</max>
+            <resolution>0.02</resolution>
+          </range>
+          <noise>
+            <type>gaussian</type>
+            <mean>0.0</mean>
+            <stddev>0.01</stddev>
+          </noise>
+        </ray>
+        <plugin name="gazebo_ros_head_rplidar_controller" filename="libgazebo_ros_laser.so">
+          <topicName>scan</topicName>
+        <frameName>$(arg robot_name)/laser_frame_link</frameName>
+        </plugin>
+      </sensor>
+    </gazebo>
   </xacro:if>
 </robot>
