Commit message: ADD: updated model with Create3 and Kobuki, sensors are now working

File: urdf/arms/mobile_wx250s.urdf.xacro (robot description, xacro)
@@ -1,10 +1,4 @@
 <?xml version="1.0"?>
 <robot name="mobile_wx250s" xmlns:xacro="http://ros.org/wiki/xacro">
-  <joint name="arm_base_link_joint" type="fixed">
-    <axis xyz="0 0 0"/>
-    <origin rpy="0 0 0" xyz="0.097277 0 0.0095"/>
-    <parent link="$(arg robot_name)/plate_link"/>
-    <child link="$(arg robot_name)/arm_base_link"/>
-  </joint>
   <link name="$(arg robot_name)/arm_base_link">
     <visual>
@@ -410,7 +404,5 @@
         <child link="$(arg robot_name)/right_finger_link"/>
         <dynamics friction="0.1"/>
-        <xacro:unless value="$(arg load_gazebo_configs)">
-          <mimic joint="left_finger" multiplier="-1" offset="0"/>
-        </xacro:unless>
+        <mimic joint="left_finger" multiplier="-1" offset="0"/>
       </joint>
       <transmission name="trans_right_finger">

File: urdf/locobot.urdf.xacro (robot description, xacro)
@@ -1,18 +1,16 @@
 <?xml version="1.0" ?>
 <robot name="locobot" xmlns:xacro="http://ros.org/wiki/xacro">
-  <xacro:arg name="arm_model" default="mobile_wx250s"/>
-  <xacro:arg name="robot_model" default="mobile_wx250s"/>
-  <xacro:arg name="robot_name" default="locobot"/>
-  <xacro:arg name="show_lidar" default="true"/>
-  <xacro:arg name="show_gripper_bar" default="true"/>
-  <xacro:arg name="show_gripper_fingers" default="true"/>
-  <xacro:arg name="external_urdf_loc" default=""/>
-  <xacro:arg name="load_gazebo_configs" default="false"/>
-  <xacro:property name="arm_type" value="$(arg arm_model)"/>
-  <xacro:property name="urdf_loc" value="$(arg external_urdf_loc)"/>
-  <xacro:property name="pi_offset" value="0.00001"/>
-  <xacro:if value="$(arg load_gazebo_configs)">
-    <xacro:include filename="$(find locobot_simulation)/config/locobot_configs.gazebo"/>
-  </xacro:if>
+  <xacro:arg name="arm_model"             default=""/>
+  <xacro:arg name="robot_model"           default=""/>
+  <xacro:arg name="base_model"            default=""/>
+  <xacro:arg name="robot_name"            default=""/>
+  <xacro:arg name="show_lidar"            default="true"/>
+  <xacro:arg name="show_gripper_bar"      default="true"/>
+  <xacro:arg name="show_gripper_fingers"  default="true"/>
+  <xacro:arg name="external_urdf_loc"     default=""/>
+  <xacro:property name="arm_type"         value="$(arg arm_model)"/>
+  <xacro:property name="base_type"        value="$(arg base_model)"/>
+  <xacro:property name="urdf_loc"         value="$(arg external_urdf_loc)"/>
+  <xacro:property name="pi_offset"        value="0.00001"/>
   <xacro:if value="${urdf_loc != ''}">
     <xacro:include filename="${urdf_loc}"/>
@@ -21,542 +19,170 @@
     <texture filename="package://locobot_simulation/meshes/interbotix_black.png"/>
   </material>
-    <!-- ********************************** Kobuki ********************************** -->
+  <xacro:include filename="$(find locobot_simulation)/urdf/plate.urdf.xacro" />
+  <xacro:include filename="$(find locobot_simulation)/urdf/lidar.urdf.xacro" />
+  <xacro:include filename="$(find locobot_simulation)/urdf/battery.urdf.xacro" />
+  <xacro:include filename="$(find locobot_simulation)/urdf/arm_cradle.urdf.xacro" />
+  <xacro:include filename="$(find locobot_simulation)/urdf/camera_tower.urdf.xacro" />
+  <xacro:include filename="$(find locobot_simulation)/urdf/pan_and_tilt.urdf.xacro" />
   <link name="$(arg robot_name)/base_footprint"/>
-  <joint name="base_joint" type="fixed">
-    <origin rpy="0 0 0" xyz="0 0 0.0102"/>
-    <parent link="$(arg robot_name)/base_footprint"/>
-    <child link="$(arg robot_name)/base_link"/>
-  </joint>
-  <link name="$(arg robot_name)/base_link">
-    <visual>
-      <origin rpy="0 0 0" xyz="0.001 0 0.05199"/>
-      <geometry>
-        <mesh filename="package://locobot_simulation/meshes/locobot_meshes/locobot_main_body.dae"/>
-      </geometry>
-    </visual>
-    <collision>
-      <origin rpy="0 0 0" xyz="0.0 0 0.05949"/>
-      <geometry>
-        <cylinder length="0.10938" radius="0.178"/>
-      </geometry>
-    </collision>
-    <inertial>
-      <origin rpy="0 0 0" xyz="0.01 0 0"/>
-      <mass value="2.4"/>
-      <inertia ixx="0.019995" ixy="0.0" ixz="0.0" iyy="0.019995" iyz="0.0" izz="0.03675"/>
-    </inertial>
-  </link>
-  <joint name="wheel_left_joint" type="continuous">
-    <axis xyz="0 0 1"/>
-    <origin rpy="-1.57079632679 0 0" xyz="0.00 0.115 0.0250"/>
-    <parent link="$(arg robot_name)/base_link"/>
-    <child link="$(arg robot_name)/wheel_left_link"/>
-  </joint>
-  <transmission name="trans_wheel_left_joint">
-    <type>transmission_interface/SimpleTransmission</type>
-    <joint name="wheel_left_joint">
-      <hardwareInterface>hardware_interface/EffortJointInterface</hardwareInterface>
-    </joint>
-    <actuator name="wheel_left_joint_motor">
-      <mechanicalReduction>1</mechanicalReduction>
-    </actuator>
-  </transmission>
-  <link name="$(arg robot_name)/wheel_left_link">
-    <visual>
-      <origin rpy="0 0 0" xyz="0 0 0"/>
-      <geometry>
-        <mesh filename="package://locobot_simulation/meshes/locobot_meshes/locobot_wheel.dae"/>
-      </geometry>
-    </visual>
-    <collision>
-      <geometry>
-        <cylinder length="0.0206" radius="0.0352"/>
-      </geometry>
-        <origin rpy="0 0 0" xyz="0 0 0"/>
-    </collision>
-    <inertial>
-      <origin xyz="0 0 0"/>
-      <mass value="0.01"/>
-      <inertia ixx="0.001" ixy="0.0" ixz="0.0" iyy="0.001" iyz="0.0" izz="0.001"/>
-    </inertial>
-  </link>
-  <joint name="wheel_right_joint" type="continuous">
-    <axis xyz="0 0 1"/>
-    <origin rpy="-1.57079632679 0 0" xyz="0.00 -0.115 0.0250"/>
-    <parent link="$(arg robot_name)/base_link"/>
-    <child link="$(arg robot_name)/wheel_right_link"/>
-  </joint>
-  <transmission name="trans_wheel_right_joint">
-    <type>transmission_interface/SimpleTransmission</type>
-    <joint name="wheel_right_joint">
-      <hardwareInterface>hardware_interface/EffortJointInterface</hardwareInterface>
-    </joint>
-    <actuator name="wheel_right_joint_motor">
-      <mechanicalReduction>1</mechanicalReduction>
-    </actuator>
-  </transmission>
-  <link name="$(arg robot_name)/wheel_right_link">
-    <visual>
-      <origin rpy="0 0 0" xyz="0 0 0"/>
-      <geometry>
-        <mesh filename="package://locobot_simulation/meshes/locobot_meshes/locobot_wheel.dae"/>
-      </geometry>
-    </visual>
-    <collision>
-      <origin rpy="0 0 0" xyz="0 0 0"/>
-      <geometry>
-        <cylinder length="0.0206" radius="0.0350"/>
-      </geometry>
-    </collision>
-    <inertial>
-      <origin xyz="0 0 0"/>
-      <mass value="0.01"/>
-      <inertia ixx="0.001" ixy="0.0" ixz="0.0" iyy="0.001" iyz="0.0" izz="0.001"/>
-    </inertial>
-  </link>
-  <joint name="caster_front_joint" type="fixed">
-    <origin rpy="-1.57079632679 0 0" xyz="0.115 0.0 0.007"/>
-    <parent link="$(arg robot_name)/base_link"/>
-    <child link="$(arg robot_name)/caster_front_link"/>
-  </joint>
-  <link name="$(arg robot_name)/caster_front_link">
-    <collision>
-      <origin rpy="0 0 0" xyz="0 0 0"/>
-      <geometry>
-        <cylinder length="0.0176" radius="0.017"/>
-      </geometry>
-    </collision>
-    <inertial>
-      <origin xyz="0 0 0"/>
-      <mass value="0.01"/>
-      <inertia ixx="0.001" ixy="0.0" ixz="0.0" iyy="0.001" iyz="0.0" izz="0.001"/>
-    </inertial>
-  </link>
-  <joint name="caster_back_joint" type="fixed">
-    <origin rpy="-1.57079632679 0 0" xyz="-0.135 0.0 0.009"/>
-    <parent link="$(arg robot_name)/base_link"/>
-    <child link="$(arg robot_name)/caster_back_link"/>
-  </joint>
-  <link name="$(arg robot_name)/caster_back_link">
-    <collision>
-      <origin rpy="0 0 0" xyz="0 0 0"/>
-      <geometry>
-        <cylinder length="0.0176" radius="0.017"/>
-      </geometry>
-    </collision>
-    <inertial>
-      <origin xyz="0 0 0"/>
-      <mass value="0.01"/>
-      <inertia ixx="0.001" ixy="0.0" ixz="0.0" iyy="0.001" iyz="0.0" izz="0.001"/>
-    </inertial>
-  </link>
-  <joint name="gyro_joint" type="fixed">
-    <origin rpy="0 0 0" xyz="0.056 0.062 0.0202"/>
-    <parent link="$(arg robot_name)/base_link"/>
-    <child link="$(arg robot_name)/gyro_link"/>
-  </joint>
-  <link name="$(arg robot_name)/gyro_link">
-    <inertial>
-      <origin rpy="0 0 0" xyz="0 0 0"/>
-      <mass value="0.001"/>
-      <inertia ixx="0.0001" ixy="0" ixz="0" iyy="0.000001" iyz="0" izz="0.0001"/>
-    </inertial>
-  </link>
-  <joint name="cliff_sensor_left_joint" type="fixed">
-    <origin rpy="0 1.57079632679 0" xyz="0.08734 0.13601 0.0214"/>
-    <parent link="$(arg robot_name)/base_link"/>
-    <child link="$(arg robot_name)/cliff_sensor_left_link"/>
-  </joint>
-  <link name="$(arg robot_name)/cliff_sensor_left_link">
-    <inertial>
-      <mass value="0.0001"/>
-      <origin xyz="0 0 0"/>
-      <inertia ixx="0.0001" ixy="0.0" ixz="0.0" iyy="0.0001" iyz="0.0" izz="0.0001"/>
-    </inertial>
-  </link>
-  <joint name="cliff_sensor_right_joint" type="fixed">
-    <origin rpy="0 1.57079632679 0" xyz="0.085 -0.13601 0.0214"/>
-    <parent link="$(arg robot_name)/base_link"/>
-    <child link="$(arg robot_name)/cliff_sensor_right_link"/>
-  </joint>
-  <link name="$(arg robot_name)/cliff_sensor_right_link">
-    <inertial>
-      <origin xyz="0 0 0"/>
-      <mass value="0.0001"/>
-      <inertia ixx="0.0001" ixy="0.0" ixz="0.0" iyy="0.0001" iyz="0.0" izz="0.0001"/>
-    </inertial>
-  </link>
-  <joint name="cliff_sensor_front_joint" type="fixed">
-    <origin rpy="0 1.57079632679 0" xyz="0.156 0.00 0.0214"/>
-    <parent link="$(arg robot_name)/base_link"/>
-    <child link="$(arg robot_name)/cliff_sensor_front_link"/>
-  </joint>
-  <link name="$(arg robot_name)/cliff_sensor_front_link">
-    <inertial>
-      <mass value="0.0001"/>
-      <origin xyz="0 0 0"/>
-      <inertia ixx="0.0001" ixy="0.0" ixz="0.0" iyy="0.0001" iyz="0.0" izz="0.0001"/>
-    </inertial>
-  </link>
-    <!-- ********************************** Bottom Plate and Arm ********************************** -->
-  <joint name="plate" type="fixed">
-    <origin rpy="0 0 0" xyz="0.0 0 0.08825"/>
-    <parent link="$(arg robot_name)/base_link"/>
-    <child link="$(arg robot_name)/plate_link"/>
-  </joint>
-  <link name="$(arg robot_name)/plate_link">
-    <visual>
-      <origin rpy="0 0 0" xyz="0 0 0"/>
-      <geometry>
-        <mesh filename="package://locobot_simulation/meshes/locobot_meshes/locobot_base_plate.stl" scale="0.001 0.001 0.001"/>
-      </geometry>
-      <material name="interbotix_black"/>
-    </visual>
-    <collision>
-      <origin rpy="0 0 0" xyz="0 0 0"/>
-      <geometry>
-        <mesh filename="package://locobot_simulation/meshes/locobot_meshes/locobot_base_plate.stl" scale="0.001 0.001 0.001"/>
-      </geometry>
-    </collision>
-    <inertial>
-      <origin rpy="0 0 0" xyz="0.050816 0 0.00475"/>
-      <mass value="0.571995"/>
-      <inertia ixx="0.003115" ixy="0" ixz="0" iyy="0.001813" iyz="0" izz="0.004919"/>
-    </inertial>
-  </link>
-  <xacro:if value="${arm_type != 'mobile_base'}">
-    <xacro:include filename="$(find locobot_simulation)/urdf/$(arg arm_model).urdf.xacro"/>
-    <xacro:if value="${arm_type == 'mobile_wx200'}">
-      <joint name="arm_cradle" type="fixed">
-         <axis xyz="0 0 0"/>
-         <origin rpy="0 0 0" xyz="0.0215 0 0.1195"/>
-         <parent link="$(arg robot_name)/camera_tower_link"/>
-         <child link="$(arg robot_name)/arm_cradle_link"/>
-      </joint>
-     <link name="$(arg robot_name)/arm_cradle_link">
-       <visual>
-         <origin rpy="0 0 0" xyz="0 0 0"/>
-         <geometry>
-           <mesh filename="package://locobot_simulation/meshes/locobot_meshes/locobot_arm_cradle.stl" scale="0.001 0.001 0.001"/>
-         </geometry>
-         <material name="interbotix_black"/>
-       </visual>
-       <collision>
-         <origin rpy="0 0 0" xyz="0 0 0"/>
-         <geometry>
-           <mesh filename="package://locobot_simulation/meshes/locobot_meshes/locobot_arm_cradle.stl" scale="0.001 0.001 0.001"/>
-         </geometry>
-       </collision>
-       <inertial>
-         <origin rpy="0 0 0" xyz="0.0014389900 0 0.0098387400"/>
-         <mass value="0.017626"/>
-         <inertia ixx="0.0000046575" ixy="0" ixz="0.0000000748" iyy="0.0000018629" iyz="0" izz="0.0000046198"/>
-       </inertial>
-     </link>
-    </xacro:if>
-  </xacro:if>
-  <!-- ********************************** Battery **********************************  -->
-  <joint name="battery" type="fixed">
-    <origin rpy="0 0 0" xyz="-0.007 0 0.0125"/>
-    <parent link="$(arg robot_name)/plate_link"/>
-    <child link="$(arg robot_name)/battery_link"/>
-  </joint>
-  <link name="$(arg robot_name)/battery_link">
-    <visual>
-      <origin rpy="0 0 0" xyz="0 0 0"/>
-      <geometry>
-        <mesh filename="package://locobot_simulation/meshes/locobot_meshes/locobot_battery.stl" scale="0.001 0.001 0.001"/>
-      </geometry>
-      <material name="">
-        <color rgba="0.5 0.5 0.5 1"/>
-      </material>
-    </visual>
-    <collision>
-      <origin rpy="0 0 0" xyz="0 0 0"/>
-      <geometry>
-        <mesh filename="package://locobot_simulation/meshes/locobot_meshes/locobot_battery.stl" scale="0.001 0.001 0.001"/>
-      </geometry>
-    </collision>
-    <inertial>
-      <origin rpy="0 0 0" xyz="0 0 0.016"/>
-      <mass value="1.194"/>
-      <inertia ixx="0.004312" ixy="0" ixz="0" iyy="0.001908" iyz="0" izz="0.006017"/>
-    </inertial>
-  </link>
-  <!-- ********************************** Camera Tower **********************************  -->
-  <joint name="camera_tower" type="fixed">
-    <origin rpy="0 0 0" xyz="-0.023997 -0.000044 0.08823"/>
-    <parent link="$(arg robot_name)/base_link"/>
-    <child link="$(arg robot_name)/camera_tower_link"/>
-  </joint>
   <xacro:if value="${arm_type == 'mobile_wx250s'}">
-    <link name="$(arg robot_name)/camera_tower_link">
-      <visual>
-        <origin rpy="0 0 0" xyz="0 0 0"/>
-        <geometry>
-          <mesh filename="package://locobot_simulation/meshes/locobot_meshes/locobot_camera_tower_large.stl" scale="0.001 0.001 0.001"/>
-        </geometry>
-        <material name="interbotix_black"/>
-      </visual>
-      <collision>
-        <origin rpy="0 0 0" xyz="0 0 0"/>
-        <geometry>
-          <mesh filename="package://locobot_simulation/meshes/locobot_meshes/locobot_camera_tower_large_simple.stl" scale="0.001 0.001 0.001"/>
-        </geometry>
-      </collision>
-      <inertial>
-        <origin rpy="0 0 0" xyz="-0.0372211000 -0.0026114300 0.1744600000"/>
-        <mass value="2.366224"/>
-        <inertia ixx="0.0628500000" ixy="0.0002152000" ixz="0.0065630000" iyy="0.0546000000" iyz="-0.0004738000" izz="0.0179300000"/>
-      </inertial>
-    </link>
+    <xacro:property name="camera_tower_size" value="large"/>
   </xacro:if>
   <xacro:unless value="${arm_type == 'mobile_wx250s'}">
-    <link name="$(arg robot_name)/camera_tower_link">
-      <visual>
-        <origin rpy="0 0 0" xyz="0 0 0"/>
-        <geometry>
-          <mesh filename="package://locobot_simulation/meshes/locobot_meshes/locobot_camera_tower_small.stl" scale="0.001 0.001 0.001"/>
-        </geometry>
-        <material name="interbotix_black"/>
-      </visual>
-      <collision>
-        <origin rpy="0 0 0" xyz="0 0 0"/>
-        <geometry>
-          <mesh filename="package://locobot_simulation/meshes/locobot_meshes/locobot_camera_tower_small_simple.stl" scale="0.001 0.001 0.001"/>
-        </geometry>
-      </collision>
+    <xacro:property name="camera_tower_size" value="small"/>
+  </xacro:unless>
+  <xacro:if value="${base_type == 'kobuki'}">
+    <xacro:include filename="$(find locobot_simulation)/urdf/kobuki_version/locobot_kobuki.urdf.xacro"/>
+    <xacro:property name="mesh_scale" value="0.001 0.001 0.001"/>
+  </xacro:if> <!-- kobuki -->
+  <xacro:if value="${base_type == 'create3'}">
+    <xacro:include filename="$(find locobot_simulation)/urdf/create3_version/locobot_create3.urdf.xacro"/>
+    <xacro:property name="mesh_scale" value="1 1 1"/>
+  </xacro:if> <!-- create3 -->
+  <!-- ********************************** Plate **********************************  -->
+  <xacro:if value="${base_type == 'kobuki'}">
+    <xacro:plate>
+      <origin rpy="0 0 0" xyz="0.0 0 0.08825"/>
       <inertial>
-        <origin rpy="0 0 0" xyz="-0.0357703000 -0.0027068600 0.1560470000"/>
-        <mass value="2.282808"/>
-        <inertia ixx="0.0461600000" ixy="0.0002062000" ixz="0.0052560000" iyy="0.0384200000" iyz="-0.0003600000" izz="0.0169600000"/>
+        <origin rpy="0 0 0" xyz="0.050816 0 0.00475"/>
+        <mass value="0.571995"/>
+        <inertia ixx="0.003115" ixy="0" ixz="0" iyy="0.001813" iyz="0" izz="0.004919"/>
       </inertial>
-    </link>
-  </xacro:unless>
+    </xacro:plate>
+  </xacro:if> <!-- base_type == 'kobuki' -->
+  <xacro:if value="${base_type == 'create3'}">
+    <xacro:plate>
+      <origin rpy="0 0 0" xyz="0 0 0.0934"/>
+      <inertial>
+        <origin rpy="0 0 0" xyz="-0.005869 0 4.67E-03"/>
+        <mass value="0.807674"/>
+        <inertia ixx="5.27E-03" ixy="0" ixz="0" iyy="3.27E-03" iyz="0" izz="8.54E-03"/>
+      </inertial>
+    </xacro:plate>
+  </xacro:if> <!-- base_type == 'create3' -->
+  <!-- ********************************** Arm ********************************** -->
+  <xacro:if value="${arm_type != 'mobile_base'}">
+    <xacro:include filename="$(find locobot_simulation)/urdf/arms/mobile_arm.urdf.xacro"/>
+    <xacro:mobile_arm/>
+    <xacro:if value="${arm_type == 'mobile_wx200'}">
+      <xacro:if value="${base_type == 'kobuki'}">
+        <xacro:arm_cradle>
+          <origin rpy="0 0 0" xyz="0.0215 0 0.1195"/>
+        </xacro:arm_cradle>
+      </xacro:if> <!-- base_type == 'kobuki' -->
+      <xacro:if value="${base_type == 'create3'}">
+        <xacro:arm_cradle>
+          <origin rpy="0 0 0" xyz="0.037943 0 0.139"/>
+        </xacro:arm_cradle>
+      </xacro:if> <!-- base_type == 'create3' -->
+    </xacro:if> <!-- arm_type == 'mobile_wx200' -->
+  </xacro:if> <!-- arm_type != 'mobile_base' -->
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